Commit message: update reward and wheel-only policy

File: Tancho_v3/Tancho_v3.urdf (robot description, URDF)
Before this commit: robot Tancho_v3, 11 links, 10 joints
Links:
- link base_link: mass 0.348 -> 0.9469
- link calf_L: mass 0.341 -> 0.1499
- link calf_R: mass 0.341 -> 0.1499
- link thigh_L: mass 0.379 -> 0.3805
- link thigh_R: mass 0.379 -> 0.3805
- link wheel_L: mass 0.152 -> 0.0349; geometry collision mesh filename=meshes/joint_wheel_L.stl; collision mesh filename=meshes/wheel_L.stl
- link wheel_R: mass 0.152 -> 0.0349; geometry collision mesh filename=meshes/joint_wheel_R.stl; collision mesh filename=meshes/wheel_R.stl
Joints:
- joint joint_calf_L: limit lower=0 upper=3 effort=12.5 velocity=12.5663706 -> lower=0 upper=3 effort=12.5 velocity=20
- joint joint_calf_R: limit lower=0 upper=3 effort=12.5 velocity=12.5663706 -> lower=0 upper=3 effort=12.5 velocity=20
- joint joint_thigh_L: limit lower=-1.57 upper=1.57 effort=12.5 velocity=12.5663706 -> lower=-1.57 upper=1.57 effort=12.5 velocity=20
- joint joint_thigh_R: limit lower=-1.57 upper=1.57 effort=12.5 velocity=12.5663706 -> lower=-1.57 upper=1.57 effort=12.5 velocity=20
- joint joint_wheel_L: limit effort=0.45 velocity=52.3598776 -> effort=0.45 velocity=188
- joint joint_wheel_R: limit effort=0.45 velocity=52.3598776 -> effort=0.45 velocity=188

File: Tancho_v3_simready/source/tancho_v3_lab/tancho_v3_lab/assets/robots/Tancho_v3/urdf/Tancho_v3.urdf (robot description, URDF)
Before this commit: robot Tancho_v3, 11 links, 10 joints
Links:
- link base_link: mass 0.348 -> 0.9469
- link calf_L: mass 0.150 -> 0.1499
- link calf_R: mass 0.150 -> 0.1499
- link thigh_L: mass 0.379 -> 0.3805
- link thigh_R: mass 0.379 -> 0.3805
- link wheel_L: mass 0.035 -> 0.0349; geometry collision mesh filename=meshes/joint_wheel_L.stl; collision mesh filename=meshes/wheel_L.stl
- link wheel_R: mass 0.035 -> 0.0349; geometry collision mesh filename=meshes/joint_wheel_R.stl; collision mesh filename=meshes/wheel_R.stl

Commit message: checkpoint Tancho V3 physics baseline diagnostics

File: Tancho_v3/Tancho_v3.urdf (robot description, URDF)
Before this commit: robot Tancho_v3, 11 links, 10 joints
Links:
- link base_link: geometry collision box size=0.18 0.091216 0.12; visual mesh filename=meshes/base_link.stl
- link calf_L: geometry collision mesh filename=meshes/calf_L.stl; visual mesh filename=meshes/calf_L.stl
- link calf_R: geometry collision mesh filename=meshes/calf_R.stl; visual mesh filename=meshes/calf_R.stl
- link drawer: geometry collision box size=0.141298 0.065 0.054994; visual mesh filename=meshes/drawer.stl
- link pi_case: geometry collision box size=0.1036 0.025 0.0656; visual mesh filename=meshes/pi_case.stl
- link thigh_L: geometry collision box size=0.075988 0.216993 0.01; collision cylinder length=0.04 radius=0.038
- link thigh_R: geometry collision box size=0.075988 0.216993 0.01; collision cylinder length=0.04 radius=0.038
- link wheel_L: geometry collision cylinder length=0.017 radius=0.03614; visual mesh filename=meshes/wheel_L.stl
- link wheel_R: geometry collision cylinder length=0.017 radius=0.03614; visual mesh filename=meshes/wheel_R.stl
